File: brake_light.kicad_sch (KiCad schematic)
At the start: 2 parts, among them U1 US2881LUA-AAA-000-BU, U2 US2881LUA-AAA-000-BU

Commit message: first commit
Parts:
- added D1, D2, D3, D4, D5, D6: LED, symbol Device:LED
- added Q1, Q2: AO3401A, Package_TO_SOT_SMD:SOT-23, symbol Transistor_FET:AO3401A
- added R1, R2: 1k, symbol Device:R
Connections:
- net +12V: now also U1.1 (VCC), U2.1 (VCC), Q1.3 (D), Q2.3 (D), R1.1, R2.1
- net GND: now also U1.3 (GND), U2.3 (GND), D1.1 (K), D2.1 (K), D3.1 (K), D4.1 (K), D5.1 (K), D6.1 (K)
- net at U2.2 (VOUT): now also Q2.1 (G), R2.2
- net at U1.2 (VOUT): now also Q1.1 (G), R1.2
- new net LOAD: D1.2 (A), D2.2 (A), D3.2 (A), D4.2 (A), D5.2 (A), D6.2 (A), Q1.2 (S), Q2.2 (S)
Other:
- note added: "HALL"
- note added: "TAILLIGHT"

Commit message: first commit
Connections:
- net +12V: now also Q1.2 (S), Q2.2 (S); no longer Q1.3 (D), Q2.3 (D)
- net LOAD: now also Q1.3 (D), Q2.3 (D); no longer Q1.2 (S), Q2.2 (S)
Changed lines of the file:
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@@
     )
   )
-  (symbol (lib_id "Transistor_FET:AO3401A") (at 181.61 71.12 0) (unit 1)
+  (symbol (lib_id "Transistor_FET:AO3401A") (at 181.61 71.12 0) (mirror x) (unit 1)
     (in_bom yes) (on_board yes) (dnp no)
-    (property "Reference" "Q2" (at 186.055 67.31 0)
+    (property "Reference" "Q2" (at 186.055 74.93 0)
       (effects (font (size 1.27 1.27)) (justify left))
     )
-    (property "Value" "AO3401A" (at 187.96 73.025 0)
+    (property "Value" "AO3401A" (at 187.96 69.215 0)
       (effects (font (size 1.27 1.27)) (justify left) hide)
     )
-    (property "Footprint" "Package_TO_SOT_SMD:SOT-23" (at 186.69 73.025 0)
+    (property "Footprint" "Package_TO_SOT_SMD:SOT-23" (at 186.69 69.215 0)
       (effects (font (size 1.27 1.27) italic) (justify left) hide)
     )
@@
     )
   )
-  (symbol (lib_id "Transistor_FET:AO3401A") (at 148.59 71.12 0) (unit 1)
+  (symbol (lib_id "Transistor_FET:AO3401A") (at 148.59 71.12 0) (mirror x) (unit 1)
     (in_bom yes) (on_board yes) (dnp no)
-    (property "Reference" "Q1" (at 152.4 66.675 0)
+    (property "Reference" "Q1" (at 152.4 75.565 0)
       (effects (font (size 1.27 1.27)) (justify left))
     )
-    (property "Value" "AO3401A" (at 154.94 73.025 0)
+    (property "Value" "AO3401A" (at 154.94 69.215 0)
       (effects (font (size 1.27 1.27)) (justify left) hide)
     )
-    (property "Footprint" "Package_TO_SOT_SMD:SOT-23" (at 153.67 73.025 0)
+    (property "Footprint" "Package_TO_SOT_SMD:SOT-23" (at 153.67 69.215 0)
       (effects (font (size 1.27 1.27) italic) (justify left) hide)
     )

Commit message: handled layout
Parts:
- removed Q2: AO3401A, Package_TO_SOT_SMD:SOT-23, symbol Transistor_FET:AO3401A
- removed R2: 1k, symbol Device:R
- removed U2: US2881LUA-AAA-000-BU, Package_TO_SOT_SMD:SOT-23W, symbol Sensor_Magnetic:A1101ELHL
- added J1: Conn_01x03, connector:3_smd_tab, symbol Connector_Generic:Conn_01x03
- R1: footprint (none) -> Resistor_SMD:R_0805_2012Metric
- U1: value US2881LUA-AAA-000-BU -> TMAG5115
Connections:
- net +12V: now also J1.1 (Pin_1)
- net GND: now also J1.3 (Pin_3)
- net LOAD: now also J1.2 (Pin_2)
Other:
- moved on the sheet: Q1, R1
